File: Kicad/M0519SD3AE/M0519SD3AE_breakout_v1/M0519SD3AE_breakout_v1.sch (KiCad schematic (older format))
At the start: 8 parts, among them U1 M0519SD3AE

Commit message: Gave up, switch back to Eagle
Parts:
- added C?: C, symbol Device:C
- added R?: R, symbol Device:R
- added SW?: SW_Push, symbol Switch:SW_Push
Connections:
- net labels added: VREF
- wire segments 30 -> 41
Changed lines of the file:
@@
 Text Label 3550 2250 0    50   ~ 0
 RST
+$Comp
+L Device:R R?
+U 1 1 5BB2CBD4
+P 1250 2050
+F 0 "R?" H 1320 2096 50  0000 L CNN
+F 1 "R" H 1320 2005 50  0000 L CNN
+F 2 "" V 1180 2050 50  0001 C CNN
+F 3 "~" H 1250 2050 50  0001 C CNN
+	1    1250 2050
+	1    0    0    -1
+$EndComp
+$Comp
+L Device:C C?
+U 1 1 5BB2CDF4
+P 1250 2600
+F 0 "C?" H 1365 2646 50  0000 L CNN
+F 1 "C" H 1365 2555 50  0000 L CNN
+F 2 "" H 1288 2450 50  0001 C CNN
+F 3 "~" H 1250 2600 50  0001 C CNN
+	1    1250 2600
+	1    0    0    -1
+$EndComp
+$Comp
+L Switch:SW_Push SW?
+U 1 1 5BB2CF0A
+P 1550 2600
+F 0 "SW?" V 1504 2748 50  0000 L CNN
+F 1 "SW_Push" V 1595 2748 50  0000 L CNN
+F 2 "" H 1550 2800 50  0001 C CNN
+F 3 "" H 1550 2800 50  0001 C CNN
+	1    1550 2600
+	0    1    1    0
+$EndComp
+$Comp
+L power:+5V #PWR?
+U 1 1 5BB2D04D
+P 1250 1600
+F 0 "#PWR?" H 1250 1450 50  0001 C CNN
+F 1 "+5V" H 1265 1773 50  0000 C CNN
+F 2 "" H 1250 1600 50  0001 C CNN
+F 3 "" H 1250 1600 50  0001 C CNN
+	1    1250 1600
+	1    0    0    -1
+$EndComp
+$Comp
+L power:GND #PWR?
+U 1 1 5BB2D06E
+P 1250 2950
+F 0 "#PWR?" H 1250 2700 50  0001 C CNN
+F 1 "GND" H 1255 2777 50  0000 C CNN
+F 2 "" H 1250 2950 50  0001 C CNN
+F 3 "" H 1250 2950 50  0001 C CNN
+	1    1250 2950
+	1    0    0    -1
+$EndComp
+Wire Wire Line
+	1250 1600 1250 1900
+Wire Wire Line
+	1550 2400 1550 2350
+Wire Wire Line
+	1550 2350 1250 2350
+Wire Wire Line
+	1250 2350 1250 2200
+Wire Wire Line
+	1250 2450 1250 2350
+Connection ~ 1250 2350
+Wire Wire Line
+	1250 2750 1250 2850
+Wire Wire Line
+	1550 2800 1550 2850
+Wire Wire Line
+	1550 2850 1250 2850
+Connection ~ 1250 2850
+Wire Wire Line
+	1250 2850 1250 2950
+Wire Wire Line
+	1550 2350 1700 2350
+Connection ~ 1550 2350
+Text Label 1600 2350 0    50   ~ 0
+RST
+Wire Wire Line
+	3750 2350 3550 2350
+Text Label 3550 2350 0    50   ~ 0
+VREF
 $EndSCHEMATC
