File: Eagle/M0519SD3AE/M0519SD3AE_breakout_v1/M0519SD3AE_breakout_v1.sch (EAGLE design)
At the start: 16 parts, among them J1 M08, J2 M08, U1 M0159S

Commit message: made some
Parts:
- added J3, J4: M04, DRances:M04
- added JP1, JP2: (no value), DRances:M06LOCK
- added R1, R2: (no value), DRances:RESISTOR0603-RES
- added SJ1, SJ2: (no value), DRances:SJ
Connections:
- new net N$1: R1.1, SJ1.2
- new net N$5: R2.1, SJ2.2
- new net N$6: R1.2, R2.2
- new net P0.4/PWM0_CH4: U1G$1.P0.4/PWM0_CH4
- new net P0.5/PWM0_CH5: U1G$1.P0.5/PWM0_CH5
- new net P1.0/PWM1_CH0: U1G$1.P1.0/PWM1_CH0
- new net P1.1/PWM1_CH1: U1G$1.P1.1/PWM1_CH1
- new net P1.2/PWM1_CH2: U1G$1.P1.2/PWM1_CH2
- new net P1.3/PWM1_CH3: U1G$1.P1.3/PWM1_CH3
- new net P1.4/PWM1_CH4: U1G$1.P1.4/PWM1_CH4
- new net P1.5/PWM1_CH5: U1G$1.P1.5/PWM1_CH5
- new net P1.6/PWM0_BRAKE0: U1G$1.P1.6/PWM0_BRAKE0
- new net P1.7/PWM1_BRAKE0: U1G$1.P1.7/PWM1_BRAKE0
- new net P2.0/SPI2_MOSI/ACMP2_0: U1G$1.P2.0/SPI2_MOSI/ACMP2_0
- new net P2.4: U1G$1.P2.4
- new net P2.5: U1G$1.P2.5
- new net P2.6/SPI0_SS/UART1_!CTS: JP1.2, U1G$1.P2.6/SPI0_SS/UART1_!CTS
- new net P2.7/SPI0_CLK/UART1_!RTS: JP1.3, U1G$1.P2.7/SPI0_CLK/UART1_!RTS
- new net P3.0/UART0_RXD: JP2.5, U1G$1.P3.0/UART0_RXD
- new net P3.1/UART0_TXD/ACMP0_O: JP2.4, U1G$1.P3.1/UART0_TXD/ACMP0_O
- new net P3.2/INT0: U1G$1.P3.2/INT0
- new net P3.4/TM0/I2C0_SDA: J4.2, U1G$1.P3.4/TM0/I2C0_SDA
- new net P3.5/TM1/I2C0_SCL: J4.3, U1G$1.P3.5/TM1/I2C0_SCL
- new net P5.0/SPI0_MOSI/UART0_!RTS: JP2.3, U1G$1.P5.0/SPI0_MOSI/UART0_!RTS
- new net P5.1/SPI0_MISO/UART0_!CTS: JP2.2, U1G$1.P5.1/SPI0_MISO/UART0_!CTS
- new net P5.2/SPI2_MISO/ACMP1_O: U1G$1.P5.2/SPI2_MISO/ACMP1_O
- new net P5.3/SPI2_CLK: U1G$1.P5.3/SPI2_CLK
- new net P5.4/SPI2_SS: U1G$1.P5.4/SPI2_SS
- new net P5.6/PWM2_CH0: U1G$1.P5.6/PWM2_CH0
- new net P5.7/PWM2_CH1: U1G$1.P5.7/PWM2_CH1
- new net P6.0/ADC0_CH0: U1G$1.P6.0/ADC0_CH0
- new net P6.1/ADC0_CH1: U1G$1.P6.1/ADC0_CH1
- new net P6.2/ADC0_CH2: U1G$1.P6.2/ADC0_CH2
- new net P6.3/ADC0_CH3: U1G$1.P6.3/ADC0_CH3
- new net P6.4/ADC0_CH4/ACMP1_N: U1G$1.P6.4/ADC0_CH4/ACMP1_N
- new net P6.5/ADC0_CH5/ACMP1_P: U1G$1.P6.5/ADC0_CH5/ACMP1_P
- new net P6.6/ADC0_CH6: U1G$1.P6.6/ADC0_CH6
- new net P6.7/ADC0_CH7: U1G$1.P6.7/ADC0_CH7
- new net P7.0/ADC1_CH0: U1G$1.P7.0/ADC1_CH0
- new net P7.1/ADC1_CH1: U1G$1.P7.1/ADC1_CH1
- new net P7.2/ADC1_CH2: U1G$1.P7.2/ADC1_CH2
- new net P7.3/ADC1_CH3: U1G$1.P7.3/ADC1_CH3
- new net P7.4/ADC1_CH4/ACMP2_N: U1G$1.P7.4/ADC1_CH4/ACMP2_N
- new net P7.5/ADC1_CH5/ACMP2_P: U1G$1.P7.5/ADC1_CH5/ACMP2_P
- new net P7.6/ADC1_CH6: U1G$1.P7.6/ADC1_CH6
- new net P7.7/ADC1_CH7: U1G$1.P7.7/ADC1_CH7
- new net P8.0/OP0_P: U1G$1.P8.0/OP0_P
- new net P8.1/OP0_N: U1G$1.P8.1/OP0_N
- new net P8.2/OP0_O: U1G$1.P8.2/OP0_O
- new net P9.0/OP1_O: U1G$1.P9.0/OP1_O
- new net P9.1/OP1_N: U1G$1.P9.1/OP1_N
- new net P9.2/OP1_P: U1G$1.P9.2/OP1_P
- new net PA.0/UART1_TXD/I2C0_SDA: J3.2, JP1.4, U1G$1.PA.0/UART1_TXD/I2C0_SDA
- new net PA.1/UART1_RXD/I2C0_SCL: J3.3, JP1.5, U1G$1.PA.1/UART1_RXD/I2C0_SCL
- net +5V: now also J3.1, J4.1, JP1.1, JP2.1
- net GND: now also J3.4, J4.4, JP1.6, JP2.6
Other:
- note added: "UART0"
- note added: "UART1"
